File: Eagle/board.brd (EAGLE design)
At the start: 49.5 x 50.5 mm, 14 parts, among them J1 5.5x2.1mm Barrel

Commit message: Updated file structure
Parts:
- moved 5REGCAP 0.25 mm to (12.7, 23.9)
- renumbered J1 to POWJACK
Changed lines of the file:
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@@
 <attribute name="VALUE" x="6.8326" y="18.6944" size="0.9906" layer="27" ratio="10" rot="R90"/>
 </element>
-<element name="5REGCAP" library="capacitor-wima" library_urn="urn:adsk.eagle:library:116" package="C5B2.5" package3d_urn="urn:adsk.eagle:package:5426/1" value="1000uf" x="12.7" y="23.622">
-<attribute name="NAME" x="8.89" y="24.892" size="1.27" layer="25" ratio="10"/>
-<attribute name="VALUE" x="10.414" y="21.59" size="1.27" layer="27" ratio="10"/>
+<element name="5REGCAP" library="capacitor-wima" library_urn="urn:adsk.eagle:library:116" package="C5B2.5" package3d_urn="urn:adsk.eagle:package:5426/1" value="1000uf" x="12.7" y="23.876">
+<attribute name="NAME" x="8.89" y="25.146" size="1.27" layer="25" ratio="10"/>
+<attribute name="VALUE" x="10.414" y="21.844" size="1.27" layer="27" ratio="10"/>
 </element>
 <element name="3VOLTREG" library="LD1117V33" package="LD1117V33" value="LD1117V33" x="21.59" y="30.48" rot="R270">
@@
 </element>
 <element name="SERVOOUT" library="pinhead" library_urn="urn:adsk.eagle:library:325" package="1X03" package3d_urn="urn:adsk.eagle:package:22458/2" value="" x="29.21" y="-8.89">
-<attribute name="NAME" x="25.3238" y="-7.0612" size="1.27" layer="25" ratio="10"/>
+<attribute name="NAME" x="25.0698" y="-7.3152" size="1.27" layer="25" ratio="10"/>
 <attribute name="VALUE" x="25.4" y="-12.065" size="1.27" layer="27"/>
 </element>
-<element name="J1" library="SparkFun-Connectors" package="POWER_JACK_SMD" value="5.5x2.1mm Barrel" x="11.43" y="-3.81">
-<attribute name="NAME" x="15.5702" y="-1.016" size="0.6096" layer="25" font="vector" ratio="20"/>
+<element name="POWJACK" library="SparkFun-Connectors" package="POWER_JACK_SMD" value="5.5x2.1mm Barrel" x="11.43" y="-3.81">
+<attribute name="NAME" x="14.0462" y="-1.524" size="0.6096" layer="25" font="vector" ratio="20"/>
 <attribute name="PROD_ID" value="CONN-08106" x="11.43" y="-3.81" size="1.778" layer="27" display="off"/>
 <attribute name="SF_ID" value="PRT-12748" x="11.43" y="-3.81" size="1.778" layer="27" display="off"/>
-<attribute name="VALUE" x="15.24" y="-7.112" size="0.6096" layer="27" font="vector" ratio="20"/>
+<attribute name="VALUE" x="12.446" y="-7.112" size="0.6096" layer="27" font="vector" ratio="20"/>
 </element>
 <element name="TRANOUT" library="transistor" library_urn="urn:adsk.eagle:library:402" package="TO220" package3d_urn="urn:adsk.eagle:package:29897/1" value="TIP122" x="33.02" y="0" rot="R270">
-<attribute name="NAME" x="38.227" y="3.81" size="1.778" layer="25" ratio="10" rot="R270"/>
-<attribute name="VALUE" x="35.56" y="3.937" size="1.778" layer="27" ratio="10" rot="R270"/>
+<attribute name="NAME" x="36.957" y="5.588" size="1.778" layer="25" ratio="10" rot="R270"/>
+<attribute name="VALUE" x="34.798" y="3.683" size="1.778" layer="27" ratio="10" rot="R270"/>
 </element>
 <element name="OUTREST" library="eagle-ltspice" library_urn="urn:adsk.eagle:library:217" package="0207/10" package3d_urn="urn:adsk.eagle:package:13275/1" value="1000" x="30.48" y="7.62">
@@
 <contactref element="5VOLTREG" pad="1"/>
 <contactref element="BATCAP" pad="1"/>
-<contactref element="J1" pad="VIN0"/>
+<contactref element="POWJACK" pad="VIN0"/>
 <wire x1="11.43" y1="1.89" x2="11.43" y2="6.35" width="0.254" layer="1"/>
 <wire x1="11.43" y1="6.35" x2="11.02" y2="6.76" width="0.254" layer="1"/>
@@
 <contactref element="3REGOUTCAP" pad="2"/>
 <contactref element="SERVOOUT" pad="1"/>
-<contactref element="J1" pad="GND"/>
+<contactref element="POWJACK" pad="GND"/>
 <polygon width="0.254" layer="1">
 <vertex x="0" y="38.6588"/>
@@
 <contactref element="TRANOUT" pad="3"/>
 <contactref element="MICROCONT" pad="GND"/>
+<wire x1="26.67" y1="-8.89" x2="26.67" y2="-2.54" width="0" layer="19" extent="1-1"/>
+<wire x1="12.7" y1="33.02" x2="15.24" y2="23.876" width="0" layer="19" extent="1-1"/>
 </signal>
 <signal name="N$3">
@@
 <contactref element="3REGCAP" pad="1"/>
 <contactref element="SERVOOUT" pad="2"/>
-<wire x1="10.16" y1="23.622" x2="6.858" y2="23.622" width="0.254" layer="1"/>
-<wire x1="6.35" y1="24.13" x2="6.858" y2="23.622" width="0.254" layer="1"/>
+<wire x1="10.16" y1="23.876" x2="6.604" y2="23.876" width="0.254" layer="1"/>
+<wire x1="6.604" y1="23.876" x2="6.35" y2="24.13" width="0.254" layer="1"/>
 <wire x1="7.04" y1="11.86" x2="5.08" y2="13.82" width="0.254" layer="1"/>
 <wire x1="5.08" y1="13.82" x2="5.08" y2="22.86" width="0.254" layer="1"/>
